File: 8bit-computer.kicad_pcb (KiCad board)
At the start: 2 copper layers, 46 parts, among them J1 Alim, SW1 Clock step, SW2 Mode sel, U1 LM2576-5.0WT, U2 NE555P, U3 74LS00, U4 74LS00, U5 NE555P, U6 NE555P

Commit message: 🚧 replace power supply with USB-C socket
Parts:
- removed C2: 1m, Capacitor_THT:CP_Radial_D13.0mm_P5.00mm
- removed D2: Red, LED_THT:LED_D5.0mm
- removed L1: 330µ, Inductor_THT:L_Toroid_Horizontal_D32.5mm_P30.00mm_Bourns_2300
- removed REF**: MountingHole_3.2mm_M3, MountingHole:MountingHole_3.2mm_M3
- removed U1: LM2576-5.0WT, Package_TO_SOT_THT:TO-220-5_Vertical
- added J2: LED_ON, Connector_PinHeader_2.54mm:PinHeader_1x02_P2.54mm_Vertical, F.Cu at (66.7, 40.0)
- added MH1: MountingHole_3.2mm_M3, MountingHole:MountingHole_3.2mm_M3, F.Cu at (21.0, 21.0)
- added MH2: MountingHole_3.2mm_M3, MountingHole:MountingHole_3.2mm_M3, F.Cu at (282.6, 21.0)
- added MH3: MountingHole_3.2mm_M3, MountingHole:MountingHole_3.2mm_M3, F.Cu at (21.0, 230.5)
- added MH4: MountingHole_3.2mm_M3, MountingHole:MountingHole_3.2mm_M3, F.Cu at (282.6, 230.5)
- added R15: 10K, Resistor_THT:R_Axial_DIN0204_L3.6mm_D1.6mm_P5.08mm_Horizontal, F.Cu at (42.5, 19.7)
- added SW3: ON/OFF, Custom:MC8MSLP1B06VS2QES, F.Cu at (29.2, 31.1)
- C1: value 100µ -> 1m; footprint Capacitor_THT:CP_Radial_D6.3mm_P2.50mm -> Capacitor_THT:CP_Radial_D13.0mm_P5.00mm
- D1: value 1N5822 -> Red; footprint Diode_THT:D_DO-201AD_P15.24mm_Horizontal -> LED_THT:LED_D5.0mm
- J1: value Alim -> Power connector; footprint Connector_BarrelJack:BarrelJack_GCT_DCJ200-10-A_Horizontal -> Connector_USB:USB_C_Receptacle_GCT_USB4085
- R1: value 10K -> 1K
- SW2: value Mode sel -> Clock mode
- moved TP3 95.9 mm to (97.2, 24.1)
- moved TP4 89.0 mm to (108.0, 24.1)
- moved R1 84.6 mm to (109.2, 56.5), turned to 180 degrees
- moved R8 80.1 mm to (111.8, 24.1), turned to 90 degrees
- moved D4 77.4 mm to (115.6, 21.6)
- moved R11 59.8 mm to (64.8, 43.8), turned to -90 degrees
- moved D3 55.7 mm to (69.2, 34.3)
- moved R5 55.7 mm to (94.0, 31.1)
- moved R9 55.7 mm to (71.5, 40.0)
- moved SW2 55.7 mm to (57.1, 24.1)
- moved C10 55.7 mm to (116.8, 29.2)
- moved C11 55.7 mm to (80.0, 22.2)
- moved C12 55.7 mm to (65.4, 22.2)
- moved C3 55.7 mm to (90.8, 32.4)
- moved C4 55.7 mm to (76.2, 32.4)
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Connections:
- net /Clock/Clk_Sel renamed /Clock/Mode
- C1 pad 1: Net-(C1-Pad1) -> VCC
- D1 pad 2: GND -> VCC
- R1 pad 1: Net-(D2-Pad1) -> /Clock/HLT
- R11 pad 1: GND -> /Clock/LEDs
- R6 pad 1: GND -> /Clock/LEDs
- U3 pad 12: GND -> /Clock/HLT
- U3 pad 13: GND -> /Clock/HLT
Routing:
- net GND: track 276.9 -> 5.53 mm
- net VCC: track 71.1 -> 0.00 mm
- net /Clock/Clk_M: track 0.00 -> 51.3 mm
- net /Clock/Mode: track 0.00 -> 44.6 mm
- net ~{CLK}: track 0.00 -> 44.3 mm
- net Net-(C5-Pad1): track 0.00 -> 44.2 mm
- net Net-(R7-Pad2): track 0.00 -> 40.1 mm
- net CLK: track 0.00 -> 39.3 mm
- net /Clock/Clk_A: track 0.00 -> 33.0 mm
- net Net-(D1-Pad1): track 37.1 -> 6.13 mm
- net Net-(R13-Pad1): track 5.72 -> 36.7 mm
- net Net-(R2-Pad2): track 0.00 -> 27.8 mm
- net Net-(R12-Pad2): track 5.72 -> 32.6 mm
- net /Clock/HLT: track 0.00 -> 24.9 mm
- net Net-(U3-Pad8): track 0.00 -> 21.8 mm
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- added copper zone on In2.Cu, net GND
- added copper zone on In1.Cu, net VCC
Other:
- board outline added: 270.5 x 218.4 mm
- copper layers 2 -> 4
- board text added: "Clock"
- board text added: "Power"
